Commit message: changes

File: control_ws/src/three_wheel/description/urdf/three_wheel_description.urdf.xacro (robot description, xacro)
@@ -15,10 +15,4 @@
   <xacro:property name="caster_wheel_radius" value="0.015" />
   <xacro:property name="z_offset" value="-${base_height/2}" /> <!-- Space btw top of beam and the each joint -->
-  <link name="base_footprint" />    <!-- set base link name -->
-  <joint name="footprint_base_joint" type="fixed">     <!-- set joint name and type-->
-      <parent link="base_footprint" />
-      <child link="base_link" />
-      <origin xyz="0 0 ${(2 * wheel_radius) + (base_height / 2.0)}" rpy="0 0 0" />
-  </joint>
   <!-- Base Link -->
   <link name="base_link">
@@ -57,5 +51,5 @@
         <origin xyz="0 0 0" rpy="${PI/2} 0 0"/>
         <geometry>
-          <cylinder length="${wheel_len}" radius="${wheel_radius}"/>
+          <sphere radius="${wheel_radius}"/>
         </geometry>
       </collision>
@@ -63,5 +57,5 @@
         <origin xyz="0 0 0" rpy="${PI/2} 0 0"/>
         <geometry>
-          <cylinder length="${wheel_len}" radius="${wheel_radius}"/>
+          <sphere radius="${wheel_radius}"/>
         </geometry>
         <material name="black"/>
@@ -71,7 +65,7 @@
         <mass value="${wheel_mass}"/>
         <inertia
-          ixx="${wheel_mass / 12.0 * (3*wheel_radius*wheel_radius + wheel_len*wheel_len)}" ixy="0.0" ixz="0.0"
-          iyy="${wheel_mass / 12.0 * (3*wheel_radius*wheel_radius + wheel_len*wheel_len)}" iyz="0.0"
-          izz="${wheel_mass / 2.0 * wheel_radius*wheel_radius}"/>
+          ixx="${wheel_mass * 0.4 * (wheel_radius * wheel_radius)}" ixy="0.0" ixz="0.0"
+          iyy="${wheel_mass * 0.4 * (wheel_radius * wheel_radius)}" iyz="0.0"
+          izz="${wheel_mass * 0.4 * (wheel_radius * wheel_radius)}"/>
       </inertial>
     </link>
@@ -88,5 +82,5 @@
         <origin xyz="0 0 0" rpy="${PI/2} 0 0"/>
         <geometry>
-          <cylinder length="${wheel_len}" radius="${wheel_radius}"/>
+          <sphere radius="${wheel_radius}"/>
         </geometry>
       </collision>
@@ -94,5 +88,5 @@
         <origin xyz="0 0 0" rpy="${PI/2} 0 0"/>
         <geometry>
-          <cylinder length="${wheel_len}" radius="${wheel_radius}"/>
+          <sphere radius="${wheel_radius}"/>
         </geometry>
         <material name="black"/>
@@ -102,7 +96,7 @@
         <mass value="${wheel_mass}"/>
         <inertia
-          ixx="${wheel_mass / 12.0 * (3*wheel_radius*wheel_radius + wheel_len*wheel_len)}" ixy="0.0" ixz="0.0"
-          iyy="${wheel_mass / 12.0 * (3*wheel_radius*wheel_radius + wheel_len*wheel_len)}" iyz="0.0"
-          izz="${wheel_mass / 2.0 * wheel_radius*wheel_radius}"/>
+          ixx="${wheel_mass * 0.4 * (wheel_radius * wheel_radius)}" ixy="0.0" ixz="0.0"
+          iyy="${wheel_mass * 0.4 * (wheel_radius * wheel_radius)}" iyz="0.0"
+          izz="${wheel_mass * 0.4 * (wheel_radius * wheel_radius)}"/>
         </inertial>
       </link>
@@ -119,5 +113,5 @@
         <origin xyz="0 0 0" rpy="${PI/2} 0 0"/>
         <geometry>
-          <cylinder length="${wheel_len}" radius="${wheel_radius}"/>
+          <sphere radius="${wheel_radius}"/>
         </geometry>
       </collision>
@@ -125,5 +119,5 @@
         <origin xyz="0 0 0" rpy="${PI/2} 0 0"/>
         <geometry>
-          <cylinder length="${wheel_len}" radius="${wheel_radius}"/>
+          <sphere radius="${wheel_radius}"/>
         </geometry>
         <material name="black"/>
@@ -133,7 +127,7 @@
         <mass value="${wheel_mass}"/>
         <inertia
-          ixx="${wheel_mass / 12.0 * (3*wheel_radius*wheel_radius + wheel_len*wheel_len)}" ixy="0.0" ixz="0.0"
-          iyy="${wheel_mass / 12.0 * (3*wheel_radius*wheel_radius + wheel_len*wheel_len)}" iyz="0.0"
-          izz="${wheel_mass / 2.0 * wheel_radius*wheel_radius}"/>
+          ixx="${wheel_mass * 0.4 * (wheel_radius * wheel_radius)}" ixy="0.0" ixz="0.0"
+          iyy="${wheel_mass * 0.4 * (wheel_radius * wheel_radius)}" iyz="0.0"
+          izz="${wheel_mass * 0.4 * (wheel_radius * wheel_radius)}"/>
         </inertial>
       </link>
